File: Project/Group_01.sch (EAGLE design)
At the start: 29 parts, among them J1 POWER_JACKPTH_LOCK, U1 +12v, U3 TCA9546A, U4 TMUX1208

Commit message: Final Version
Connections:
- net N$1 renamed SWITCH
- net N$10 renamed S1
- net N$11 renamed S2
- net N$12 renamed S3
- net N$13 renamed S4
- net N$14 renamed S5
- net N$15 renamed S6
- net N$16 renamed S7
- net N$17 renamed S8
- net N$2 renamed P_0.5
- net N$3 renamed P_0.4
- net N$4 renamed P_0.3
- net N$5 renamed P_0.2
- net N$6 renamed P_0.1
- net N$7 renamed P_0.0
Changed lines of the file:
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@@
 <setting verticaltext="up"/>
 </settings>
-<grid distance="0.1" unitdist="mm" unit="mm" style="lines" multiple="1" display="no" altdistance="0.01" altunitdist="inch" altunit="inch"/>
+<grid distance="0.1" unitdist="inch" unit="inch" style="lines" multiple="1" display="no" altdistance="0.01" altunitdist="inch" altunit="inch"/>
 <layers>
 <layer number="1" name="Top" color="4" fill="1" visible="no" active="no"/>
@@
 </segment>
 </net>
-<net name="N$2" class="0">
+<net name="P_0.5" class="0">
 <segment>
 <pinref part="U$2" gate="G$1" pin="P_0.5"/>
@@
 </segment>
 </net>
-<net name="N$3" class="0">
+<net name="P_0.4" class="0">
 <segment>
 <pinref part="U$2" gate="G$1" pin="P_0.4"/>
@@
 </segment>
 </net>
-<net name="N$4" class="0">
+<net name="P_0.3" class="0">
 <segment>
 <pinref part="U$2" gate="G$1" pin="P_0.3"/>
@@
 </segment>
 </net>
-<net name="N$5" class="0">
+<net name="P_0.2" class="0">
 <segment>
 <pinref part="U$2" gate="G$1" pin="P_0.2"/>
@@
 </segment>
 </net>
-<net name="N$6" class="0">
+<net name="P_0.1" class="0">
 <segment>
 <pinref part="U$2" gate="G$1" pin="P_0.1"/>
@@
 </segment>
 </net>
-<net name="N$7" class="0">
+<net name="P_0.0" class="0">
 <segment>
 <pinref part="U$2" gate="G$1" pin="P_0.0"/>
@@
 </segment>
 </net>
-<net name="N$1" class="0">
-<segment>
-<pinref part="J1" gate="G$1" pin="PWR"/>
-<pinref part="S1" gate="1" pin="P"/>
-<wire x1="147.86" y1="129.92" x2="130.08" y2="129.92" width="0.1524" layer="91"/>
+<net name="S1" class="0">
+<segment>
+<pinref part="J8" gate="G$1" pin="8"/>
+<pinref part="U4" gate="G$1" pin="S1"/>
+<wire x1="102.14" y1="71.5" x2="107.22" y2="71.5" width="0.1524" layer="91"/>
 </segment>
 </net>
@@
 </segment>
 </net>
-<net name="N$10" class="0">
-<segment>
-<pinref part="J8" gate="G$1" pin="8"/>
-<pinref part="U4" gate="G$1" pin="S1"/>
-<wire x1="102.14" y1="71.5" x2="107.22" y2="71.5" width="0.1524" layer="91"/>
-</segment>
-</net>
-<net name="N$11" class="0">
+<net name="S2" class="0">
 <segment>
 <pinref part="J8" gate="G$1" pin="7"/>
@@
 </segment>
 </net>
-<net name="N$12" class="0">
+<net name="S3" class="0">
 <segment>
 <pinref part="J8" gate="G$1" pin="6"/>
@@
 </segment>
 </net>
-<net name="N$13" class="0">
+<net name="S4" class="0">
 <segment>
 <pinref part="J8" gate="G$1" pin="5"/>
@@
 </segment>
 </net>
-<net name="N$14" class="0">
+<net name="S5" class="0">
 <segment>
 <pinref part="J8" gate="G$1" pin="4"/>
@@
 </segment>
 </net>
-<net name="N$15" class="0">
+<net name="S6" class="0">
 <segment>
 <pinref part="J8" gate="G$1" pin="3"/>
@@
 </segment>
 </net>
-<net name="N$16" class="0">
+<net name="S7" class="0">
 <segment>
 <pinref part="J8" gate="G$1" pin="2"/>
@@
 </segment>
 </net>
-<net name="N$17" class="0">
+<net name="S8" class="0">
 <segment>
 <pinref part="J8" gate="G$1" pin="1"/>
@@
 </segment>
 </net>
+<net name="SWITCH" class="0">
+<segment>
+<pinref part="J1" gate="G$1" pin="PWR"/>
+<pinref part="S1" gate="1" pin="P"/>
+<wire x1="147.86" y1="129.92" x2="130.08" y2="129.92" width="0.1524" layer="91"/>
+</segment>
+</net>
