File: Project/Group_01.brd (EAGLE design)
At the start: 71.1 x 54.3 mm, 29 parts, among them J1 POWER_JACKPTH_LOCK, U1 +12v, U3 TCA9546A, U4 TMUX1208

Commit message: Final Version
Parts:
- moved C3 1.55 mm to (49.5, 11.4)
- moved C1 0.94 mm to (25.2, 4.87)
Connections:
- net N$1 renamed SWITCH
- net N$10 renamed S1
- net N$11 renamed S2
- net N$12 renamed S3
- net N$13 renamed S4
- net N$14 renamed S5
- net N$15 renamed S6
- net N$16 renamed S7
- net N$17 renamed S8
- net N$2 renamed P_0.5
- net N$3 renamed P_0.4
- net N$4 renamed P_0.3
- net N$5 renamed P_0.2
- net N$6 renamed P_0.1
- net N$7 renamed P_0.0
Routing:
- net MUX_OUT: track 28.9 -> 26.3 mm
- net GND: track 203.6 -> 204.5 mm
- net S5: track 9.94 -> 9.09 mm
- net S8: track 13.1 -> 13.7 mm
- net 5V: track 243.9 -> 244.5 mm
Other:
- board text added: "5V"
- board text added: "GND"
